Commit message: solved problems in IO_evaluator and evaluation process

File: urdf/cube/cube.urdf (robot description, URDF)
Before this commit: robot cube, 1 links, 0 joints
Links:
- link baseLink: geometry collision mesh filename=cube.obj scale=1.2 1.2 1.2; visual mesh filename=cube.obj scale=1.2 1.2 1.2

Commit message: sync, grasp diagonally

File: urdf/cube/cube.urdf (robot description, URDF)
Before this commit: robot cube, 1 links, 0 joints
Links:
- link baseLink: geometry collision mesh filename=cube.obj scale=1.5 1.2 1.2; visual mesh filename=cube.obj scale=1.5 1.2 1.2
